File: eagle/AudioLed.brd (EAGLE design)
At the start: 42.5 x 39.4 mm, 39 parts, among them Q1 8/16/20MHz, Q2 CMA-4544PF-W, U1 ATMEGA328, U2 L7805CDT-TR, U4 MAX9814TDFN14

Commit message: Fix Incorrectly Labled Capacitor
Parts:
- C13: value 0.1uF -> 33pF
Changed lines of the file:
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@@
 <attribute name="VALUE" x="1.2065" y="28.321" size="0.508" layer="27" rot="R270"/>
 </element>
-<element name="C13" library="adafruit" package="C0805" value="0.1uF" x="3.81" y="24.765" smashed="yes">
+<element name="C13" library="adafruit" package="C0805" value="33pF" x="3.81" y="24.765" smashed="yes">
 <attribute name="VALUE" x="1.651" y="23.749" size="0.508" layer="27" rot="R90"/>
 </element>
