File: eagle/AudioLed.brd (EAGLE design)
At the start: 42.5 x 39.4 mm, 39 parts, among them Q1 8/16/20MHz, Q2 CMA-4544PF-W, U1 ATMEGA328, U2 L7805CDT-TR, U4 MAX9814TDFN14

Commit message: Replace bad resonator with SparkFun Resonator
Parts:
- Q1: value 8/16/20MHz -> 16MHZ; device Testing:RESONATOR-SMD-1:1 -> SparkFun-FreqCtrl:RESONATOR-SMD
Changed lines of the file:
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@@
 <attribute name="VALUE" x="39.5732" y="11.8872" size="0.8128" layer="27" rot="R180"/>
 </element>
-<element name="Q1" library="Testing" package="RESONATOR-SMD-1:1" value="8/16/20MHz" x="19.450234375" y="17.223378125" smashed="yes" rot="R225"/>
+<element name="Q1" library="SparkFun-FreqCtrl" package="RESONATOR-SMD" value="16MHZ" x="19.450234375" y="17.223378125" smashed="yes" rot="R225">
+<attribute name="PROD_ID" value="XTAL-08900" x="19.450234375" y="17.223378125" size="1.778" layer="27" rot="R225" display="off"/>
+<attribute name="VALUE" value="16MHZ" x="19.450234375" y="17.223378125" size="1.778" layer="27" rot="R225" display="off"/>
+</element>
 <element name="U2" library="BAG" package="DPAK" value="L7805CDT-TR" x="23.114" y="29.2735" smashed="yes">
 <attribute name="VALUE" x="20.6375" y="27.9845" size="0.508" layer="27"/>
