File: eagle/AudioLed.sch (EAGLE design)
At the start: 39 parts, among them Q1 8/16/20MHz, Q2 CMA-4544PF-W, U1 ATMEGA328, U2 L7805CDT-TR, U4 MAX9814TDFN14

Commit message: Fix Incorrectly Labled Capacitor
Parts:
- C13: value 0.1uF -> 33pF
Changed lines of the file:
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@@
 <part name="C12" library="adafruit" deviceset="C-US" device="C0805" value="0.1uF"/>
 <part name="GND17" library="SparkFun" deviceset="GND" device=""/>
-<part name="C13" library="adafruit" deviceset="C-US" device="C0805" value="0.1uF"/>
+<part name="C13" library="adafruit" deviceset="C-US" device="C0805" value="33pF"/>
 <part name="GND18" library="SparkFun" deviceset="GND" device=""/>
 <part name="R7" library="adafruit" deviceset="R-US_" device="M0805" value="200K"/>
